File: schematics/multi_sensor_host/multi_sensor_host.kicad_sch (KiCad schematic)
At the start: 45 parts, among them J1 esp_rst, J2 esp_flash_wifi, J3 esp_flash_uart, J4 esp_flash_port, J6 MY_USB_B, J7 swd, P1 USB_B, P2 ~rst~, P3 bootldr, U11 stm32f405rgt6, U8 MCP73812T-420I-OT, Y1 Crystal

Commit message: a
Parts:
- removed D3, D4: LED, LED_THT:LED_D3.0mm, symbol bridge-rescue:LED
- removed J7: swd, Connector_PinHeader_1.27mm:PinHeader_1x03_P1.27mm_Vertical, symbol bridge-rescue:CONN_01X03
- removed P1: USB_B, Connectors:USB_B, symbol multi_i2c-rescue:USB_B
- removed P2: ~rst~, Connector_PinHeader_1.27mm:PinHeader_1x02_P1.27mm_Vertical, symbol bridge-rescue:CONN_01X02
- removed P3: bootldr, Connector_PinHeader_1.27mm:PinHeader_1x02_P1.27mm_Vertical, symbol bridge-rescue:CONN_01X02
- added C21: 4u7, Capacitors_SMD:C_0603, symbol multi_i2c-rescue:C
- added D3, D4, D6: LED, LED_THT:LED_D3.0mm, symbol Device:LED
- added J10: swd, symbol Connector:Conn_01x03_Pin
- added J11: stm_boot, symbol Connector:Conn_01x02_Pin
- added J5: tx, symbol Connector:Conn_01x02_Pin
- added J7: rst, symbol Connector:Conn_01x02_Pin
- added J8: rx, symbol Connector:Conn_01x02_Pin
- added J9: uart1, symbol Connector:Conn_01x04_Pin
- added R92: 1k 5%, Resistor_SMD:R_0603_1608Metric, symbol bridge-rescue:R
- added R93: 10k 5%, Resistor_SMD:R_0603_1608Metric, symbol bridge-rescue:R
- added R94, R95: 100k 5%, Resistor_SMD:R_0603_1608Metric, symbol bridge-rescue:R
- J3: value esp_flash_uart -> esp_boot
Connections:
- net i2c_scl is gone; now on net scl_host_a: U11.58 (PB6__USART1_TX)
- net i2c_sda is gone; now on net sda_host_a: U11.59 (PB7__USART1_RX)
- net pa5 is gone; now on net led-0: U11.21 (PA5)
- net pa6 is gone; now on net led-1: U11.22 (PA6)
- net pb10 is gone; now on net scl_host_b: U11.29 (PB10___USART3_TX)
- net pb11 is gone; now on net sda_host_b: U11.30 (PB11___USART3_RX)
- net spi_miso is gone; now on net shifter_clock: U11.52 (PC11__USART4_RX)
- net spi_nss is gone; now on net parallel_load: U11.50 (PA15___JTDI)
- net spi_sck is gone; now on net data_serial: U11.51 (PC10___USART4_TX)
- net vbus is gone; now on net Vbus: C10.1, J6.1 (VBUS)
- net GND: now also C21.2, D3.2 (A), D4.2 (A), D6.2 (A), J10.2 (Pin_2), J7.2 (Pin_2), J9.4 (Pin_4), R95.2
- net VDD: now also J11.1 (Pin_1), J9.3 (Pin_3), R93.1
- net boot0: now also J11.2 (Pin_2)
- net esp_rx: now also J8.1 (Pin_1)
- net led-0: no longer U11.15 (PA1)
- net led-1: no longer U11.16 (PA2)
- net swd_clk: now also J10.1 (Pin_1)
- net swd_io: now also J10.3 (Pin_3)
- net ~{mcu-rst}: now also J7.1 (Pin_1)
- net at R89.2: now also D6.1 (K)
- net Vbatt: now reaches C8.1, D1.2 (A), TP1.1, U8.3 (V_{BAT})
- net Vbatt: now also R94.1
- net batt_sense: now reaches U11.14 (PA0-WKUP)
- net batt_sense: now also C21.1, R94.2, R95.1
- net stm_rx: now reaches U11.17 (PA3)
- net stm_rx: now also J5.2 (Pin_2)
- net uart1-tx: now reaches U11.42 (PA9_USART1_TX)
- net uart1-tx: now also J9.1 (Pin_1)
- net uart1-rx: now reaches U11.43 (PA10___OTG_FS_ID/USART1_RX)
- net uart1-rx: now also J9.2 (Pin_2), R93.2
- net at R90.2: now also D3.1 (K)
- net dev_dm: no longer names the net of U11.44 (PA11___OTG_FS_DM)
- net dev_dp: no longer names the net of U11.45 (PA12___OTG_FS_DP)
- net pa4: no longer names the net of U11.20 (PA4)
- net pa7 renamed led-2
- net led-2: now also R92.1
- net pb0: no longer names the net of U11.26 (PB0)
- net pb1: no longer names the net of U11.27 (PB1)
- net pb2: no longer names the net of U11.28 (PB2)
- net pc4: no longer names the net of U11.24 (PC4)
- net pc5: no longer names the net of U11.25 (PC5)
- net spi_mosi: no longer names the net of U11.53 (PC12)
- new net: D4.1 (K), R92.2
- new net esp_tx: J5.1 (Pin_1)
- new net stm_tx: J8.2 (Pin_2), U11.16 (PA2)
- no-connect marks 24 -> 39
Other:
- moved on the sheet: C23, C24, C27, C28, C29, C30, C31, U11A, U11B

Commit message: Cannot re-save stm32f405rgt6. May be need to copy it again from the other project.
Parts:
- C10, C23, C24, C27, C28, C29, C30, C31, C4, C5, C9: symbol bridge-rescue:C -> Device:C
- C21, C3, C6, C7, C8: symbol multi_i2c-rescue:C -> Device:C
- J6: symbol bridge-rescue:MY_USB_B -> Connector:USB_B
- R83, R84, R85, R86: symbol multi_i2c-rescue:R -> Device:R
- R87, R88, R89, R90, R91, R92, R93, R94, R95: symbol bridge-rescue:R -> Device:R
- U: renamed from U11; value stm32f405rgt6 -> ~

Commit message: Fixed STM MCU symbol.
Parts:
- removed U: ~, symbol bridge-rescue:stm32f405rgt6
- added J12: DC37_Receptacle_MountingHoles, symbol Connector:DC37_Receptacle_MountingHoles
- added U10: ~, symbol stm32f405rgt6_2:STM32F405RGT6
Connections:
- net GND: now also U10.12 (VssA), U10.18 (Vss_1), U10.63 (Vss_2)
- net VDD: now also U10.1 (VBAT), U10.13 (VDDA), U10.19 (VDD_4), U10.32 (VDD_1), U10.48 (VDD_2), U10.64 (VDD_3)
- net batt_sense: now also U10.14 (PA0-WKUP)
- net boot0: now also U10.60 (BOOT0)
- net clk-in: now also U10.5 (PD0_OSC_IN)
- net clk-out: now also U10.6 (PD1_OSC_OUT)
- net data_serial: now also U10.51 (PC10___USART4_TX)
- net host_dm: now also U10.35 (PB14___OTG_HS_DM)
- net host_dp: now also U10.36 (PB15___OTG_HS_DP)
- net led-0: now also U10.21 (PA5)
- net led-1: now also U10.22 (PA6)
- net led-2: now also U10.23 (PA7)
- net parallel_load: now also U10.50 (PA15___JTDI)
- net scl_host_a: now also U10.58 (PB6__USART1_TX)
- net scl_host_b: now also U10.29 (PB10___USART3_TX)
- net sda_host_a: now also U10.59 (PB7__USART1_RX)
- net sda_host_b: now also U10.30 (PB11___USART3_RX)
- net shifter_clock: now also U10.52 (PC11__USART4_RX)
- net stm_rx: now also U10.17 (PA3)
- net stm_tx: now also U10.16 (PA2)
- net swd_clk: now also U10.49 (PA14___JTCK-SWCLK)
- net swd_io: now also U10.46 (PA13___JTMS-SWDIO)
- net uart1-rx: now also U10.43 (PA10___OTG_FS_ID/USART1_RX)
- net uart1-tx: now also U10.42 (PA9_USART1_TX)
- net ~{mcu-rst}: now also U10.7 (NRST)
- net at C28.2: now also U10.31 (Vcap_1)
- net at C29.2: now also U10.47 (Vcap_2)
Other:
- moved on the sheet: C10, C21, C23, C24, C27, C28, C29, C30, C31, C4, C5, C9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
