File: schematics/multi_sensor_host/multi_sensor_host.kicad_sch (KiCad schematic)
At the start: 84 parts, among them J1 RJ45, J10 swd, J11 stm_boot, J12 rst_cmn, J17 bm_rst, J18 RJ45, J19 RJ45, J2 RJ45, J20 RJ45, J21 RJ45, J22 RJ45, J23 RJ45, J24 RJ45, J25 RJ45, J26 RJ45, J27 RJ45, J28 RJ45, J29 RJ45, J3 bm_cfg, J30 RJ45, J4 RJ45, J5 tx, J6 MY_USB_B, J7 rst, J8 rx, J9 uart1, U12 BM71BLES1FC2-0B02AA, U8 MCP73812T-420I-OT, Y1 Crystal

Commit message: Assigned footprints. Also, just in case found a chip I2C to diff. pair.
Parts:
- C21, C22, C3, C32, C33, C34, C35, C6, C7, C8: footprint Capacitors_SMD:C_0603 -> Capacitor_SMD:C_0603_1608Metric
- D1, D2: value D_Schottky -> 1N5819; footprint (none) -> Diode_THT:D_DO-41_SOD81_P7.62mm_Horizontal
- J1, J18, J19, J2, J20, J21, J22, J23, J24, J25, J26, J27, J28, J29, J30, J4: footprint (none) -> Connector_RJ:RJ45_OST_PJ012-8P8CX_Vertical
- J10: footprint (none) -> Connector_PinHeader_2.54mm:PinHeader_1x03_P2.54mm_Vertical
- J11, J12, J17, J3, J5, J7, J8: footprint (none) -> Connector_PinHeader_2.54mm:PinHeader_1x02_P2.54mm_Vertical
- J6: footprint Connector_USB:USB_B_Horizontal -> Connector_USB:USB_B_Lumberg_2411_02_Horizontal
- J9: footprint (none) -> Connector_PinHeader_2.54mm:PinHeader_1x04_P2.54mm_Vertical
- R83, R84, R85, R86, R96, R97: footprint Resistors_SMD:R_0603 -> Capacitor_SMD:C_0603_1608Metric
- R98: footprint Resistor_SMD:R_0603_1608Metric -> Capacitor_SMD:C_0603_1608Metric
- TP1, TP2: footprint (none) -> TestPoint:TestPoint_Pad_D4.0mm
- TP3, TP4, TP5, TP6, TP7, TP8: footprint (none) -> TestPoint:TestPoint_Pad_D2.0mm
- U10: footprint (none) -> Package_QFP:LQFP-64_10x10mm_P0.5mm
- U11: value ~ -> MCP111
- U12: footprint BM71BLES1FC2_MCH -> BM71BLES1FC2_MCH:BM71BLES1FC2_MCH
- U9: value ~ -> mcp1603t-330
- Y1: footprint (none) -> Crystal:Crystal_HC52-8mm_Vertical
Changed lines of the file:
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@@
 			)
 		)
-		(property "Footprint" ""
+		(property "Footprint" "Connector_PinHeader_2.54mm:PinHeader_1x02_P2.54mm_Vertical"
 			(at 414.02 351.79 0)
 			(effects
@@
 			)
 		)
-		(property "Footprint" "Resistors_SMD:R_0603"
+		(property "Footprint" "Capacitor_SMD:C_0603_1608Metric"
 			(at 588.772 172.72 90)
 			(effects
@@
 			)
 		)
-		(property "Footprint" "Capacitors_SMD:C_0603"
+		(property "Footprint" "Capacitor_SMD:C_0603_1608Metric"
 			(at 512.7752 132.08 0)
 			(effects
@@
 			)
 		)
-		(property "Footprint" ""
+		(property "Footprint" "Connector_PinHeader_2.54mm:PinHeader_1x02_P2.54mm_Vertical"
 			(at 608.33 181.61 0)
 			(effects
@@
 			)
 		)
-		(property "Footprint" ""
+		(property "Footprint" "Connector_PinHeader_2.54mm:PinHeader_1x02_P2.54mm_Vertical"
 			(at 603.25 118.11 0)
 			(effects
@@
 			)
 		)
-		(property "Footprint" "Connector_USB:USB_B_Horizontal"
+		(property "Footprint" "Connector_USB:USB_B_Lumberg_2411_02_Horizontal"
 			(at 172.72 354.33 0)
 			(effects
@@
 			)
 		)
-		(property "Footprint" ""
+		(property "Footprint" "Connector_RJ:RJ45_OST_PJ012-8P8CX_Vertical"
 			(at 730.25 236.855 90)
 			(effects
@@
 			)
 		)
-		(property "Footprint" ""
+		(property "Footprint" "Connector_RJ:RJ45_OST_PJ012-8P8CX_Vertical"
 			(at 730.25 262.255 90)
 			(effects
@@
 			)
 		)
-		(property "Footprint" ""
+		(property "Footprint" "Connector_RJ:RJ45_OST_PJ012-8P8CX_Vertical"
 			(at 703.58 85.725 90)
 			(effects
@@
 			)
 		)
-		(property "Value" "~"
+		(property "Value" "mcp1603t-330"
 			(at 414.02 26.67 0)
 			(effects
@@
 			)
 		)
-		(property "Footprint" ""
+		(property "Footprint" "Connector_RJ:RJ45_OST_PJ012-8P8CX_Vertical"
 			(at 774.7 34.925 90)
 			(effects
@@
 			)
 		)
-		(property "Footprint" ""
+		(property "Footprint" "Package_QFP:LQFP-64_10x10mm_P0.5mm"
 			(at 323.85 367.03 0)
 			(effects
@@
 			)
 		)
-		(property "Value" "D_Schottky"
+		(property "Value" "1N5819"
 			(at 180.6575 57.15 0)
 			(effects
@@
 			)
 		)
-		(property "Footprint" ""
+		(property "Footprint" "Diode_THT:D_DO-41_SOD81_P7.62mm_Horizontal"
 			(at 180.34 60.96 0)
 			(effects
@@
 			)
 		)
-		(property "Footprint" ""
+		(property "Footprint" "Connector_PinHeader_2.54mm:PinHeader_1x02_P2.54mm_Vertical"
 			(at 566.42 181.61 0)
 			(effects
@@
 			)
 		)
-		(property "Footprint" ""
+		(property "Footprint" "TestPoint:TestPoint_Pad_D2.0mm"
 			(at 448.31 173.99 0)
 			(effects
@@
 			)
 		)
-		(property "Footprint" ""
+		(property "Footprint" "Connector_PinHeader_2.54mm:PinHeader_1x02_P2.54mm_Vertical"
 			(at 571.5 133.35 0)
 			(effects
@@
 			)
 		)
-		(property "Footprint" ""
+		(property "Footprint" "Connector_PinHeader_2.54mm:PinHeader_1x04_P2.54mm_Vertical"
 			(at 166.37 314.96 0)
 			(effects
@@
 			)
 		)
-		(property "Value" "D_Schottky"
+		(property "Value" "1N5819"
 			(at 271.78 50.4824 90)
 			(effects
@@
 			)
 		)
-		(property "Footprint" ""
+		(property "Footprint" "Diode_THT:D_DO-41_SOD81_P7.62mm_Horizontal"
 			(at 269.24 49.53 0)
 			(effects
@@
 			)
 		)
-		(property "Footprint" ""
+		(property "Footprint" "Connector_RJ:RJ45_OST_PJ012-8P8CX_Vertical"
 			(at 774.7 60.325 90)
 			(effects
@@
 			)
 		)
-		(property "Footprint" ""
+		(property "Footprint" "TestPoint:TestPoint_Pad_D2.0mm"
 			(at 448.31 168.91 0)
 			(effects
@@
 			)
 		)
-		(property "Footprint" ""
+		(property "Footprint" "Crystal:Crystal_HC52-8mm_Vertical"
 			(at 434.34 419.1 0)
 			(effects
@@
 			)
 		)
-		(property "Footprint" "Resistors_SMD:R_0603"
+		(property "Footprint" "Capacitor_SMD:C_0603_1608Metric"
 			(at 385.572 130.81 90)
 			(effects
@@
 			)
 		)
-		(property "Footprint" ""
+		(property "Footprint" "Connector_RJ:RJ45_OST_PJ012-8P8CX_Vertical"
 			(at 703.58 34.925 90)
 			(effects
@@
 			)
 		)
-		(property "Footprint" "Capacitors_SMD:C_0603"
+		(property "Footprint" "Capacitor_SMD:C_0603_1608Metric"
 			(at 520.3952 132.08 0)
 			(effects
@@
 			)
 		)
-		(property "Footprint" "Resistors_SMD:R_0603"
+		(property "Footprint" "Capacitor_SMD:C_0603_1608Metric"
 			(at 215.138 77.47 90)
 			(effects
@@
 			)
 		)
-		(property "Footprint" ""
+		(property "Footprint" "Connector_RJ:RJ45_OST_PJ012-8P8CX_Vertical"
 			(at 774.7 85.725 90)
 			(effects
@@
 			)
 		)
-		(property "Footprint" "Capacitors_SMD:C_0603"
+		(property "Footprint" "Capacitor_SMD:C_0603_1608Metric"
 			(at 248.6152 66.04 0)
 			(effects
@@
 			)
 		)
-		(property "Footprint" ""
+		(property "Footprint" "Connector_RJ:RJ45_OST_PJ012-8P8CX_Vertical"
 			(at 774.7 111.125 90)
 			(effects
@@
 			)
 		)
-		(property "Footprint" ""
+		(property "Footprint" "Package_QFP:LQFP-64_10x10mm_P0.5mm"
 			(at 73.66 384.81 0)
 			(effects
@@
 			)
 		)
-		(property "Footprint" ""
+		(property "Footprint" "TestPoint:TestPoint_Pad_D4.0mm"
 			(at 285.75 68.58 0)
 			(effects
@@
 			)
 		)
-		(property "Footprint" ""
+		(property "Footprint" "Connector_PinHeader_2.54mm:PinHeader_1x02_P2.54mm_Vertical"
 			(at 448.31 322.58 0)
 			(effects
@@
 			)
 		)
-		(property "Footprint" ""
+		(property "Footprint" "TestPoint:TestPoint_Pad_D4.0mm"
 			(at 285.75 60.96 0)
 			(effects
@@
 			)
 		)
-		(property "Footprint" "Capacitors_SMD:C_0603"
+		(property "Footprint" "Capacitor_SMD:C_0603_1608Metric"
 			(at 528.0152 132.08 0)
 			(effects
@@
 			)
 		)
-		(property "Footprint" ""
+		(property "Footprint" "Connector_PinHeader_2.54mm:PinHeader_1x03_P2.54mm_Vertical"
 			(at 424.18 292.1 0)
 			(effects
@@
 			)
 		)
-		(property "Footprint" "BM71BLES1FC2_MCH"
+		(property "Footprint" "BM71BLES1FC2_MCH:BM71BLES1FC2_MCH"
 			(at 421.64 123.19 0)
 			(effects
@@
 			)
 		)
-		(property "Footprint" "Capacitors_SMD:C_0603"
+		(property "Footprint" "Capacitor_SMD:C_0603_1608Metric"
 			(at 450.5452 39.37 0)
 			(effects
@@
 			)
 		)
-		(property "Footprint" ""
+		(property "Footprint" "Connector_RJ:RJ45_OST_PJ012-8P8CX_Vertical"
 			(at 703.58 60.325 90)
 			(effects
@@
 			)
 		)
-		(property "Footprint" "Capacitors_SMD:C_0603"
+		(property "Footprint" "Capacitor_SMD:C_0603_1608Metric"
 			(at 591.5152 193.04 0)
 			(effects
@@
 			)
 		)
-		(property "Footprint" ""
+		(property "Footprint" "Connector_RJ:RJ45_OST_PJ012-8P8CX_Vertical"
 			(at 774.7 156.845 90)
 			(effects
@@
 			)
 		)
-		(property "Footprint" ""
+		(property "Footprint" "Connector_RJ:RJ45_OST_PJ012-8P8CX_Vertical"
 			(at 730.25 313.055 90)
 			(effects
@@
 			)
 		)
-		(property "Footprint" "Resistor_SMD:R_0603_1608Metric"
+		(property "Footprint" "Capacitor_SMD:C_0603_1608Metric"
 			(at 515.112 165.1 90)
 			(effects
@@
 			)
 		)
-		(property "Footprint" "Capacitors_SMD:C_0603"
+		(property "Footprint" "Capacitor_SMD:C_0603_1608Metric"
 			(at 554.6852 144.78 0)
 			(effects
@@
 			)
 		)
-		(property "Footprint" "Capacitors_SMD:C_0603"
+		(property "Footprint" "Capacitor_SMD:C_0603_1608Metric"
 			(at 381.9652 39.37 0)
 			(effects
@@
 			)
 		)
-		(property "Footprint" ""
+		(property "Footprint" "TestPoint:TestPoint_Pad_D2.0mm"
 			(at 448.31 176.53 0)
 			(effects
@@
 			)
 		)
-		(property "Footprint" "Resistors_SMD:R_0603"
+		(property "Footprint" "Capacitor_SMD:C_0603_1608Metric"
 			(at 215.138 67.31 90)
 			(effects
@@
 			)
 		)
-		(property "Footprint" ""
+		(property "Footprint" "Connector_RJ:RJ45_OST_PJ012-8P8CX_Vertical"
 			(at 703.58 156.845 90)
 			(effects
@@
 			)
 		)
-		(property "Footprint" "Resistors_SMD:R_0603"
+		(property "Footprint" "Capacitor_SMD:C_0603_1608Metric"
 			(at 215.138 87.63 90)
 			(effects
@@
 			)
 		)
-		(property "Footprint" ""
+		(property "Footprint" "Connector_RJ:RJ45_OST_PJ012-8P8CX_Vertical"
 			(at 703.58 111.125 90)
 			(effects
@@
 			)
 		)
-		(property "Footprint" ""
+		(property "Footprint" "Connector_RJ:RJ45_OST_PJ012-8P8CX_Vertical"
 			(at 730.25 287.655 90)
 			(effects
@@
 			)
 		)
-		(property "Footprint" "Capacitors_SMD:C_0603"
+		(property "Footprint" "Capacitor_SMD:C_0603_1608Metric"
 			(at 218.1352 321.31 0)
 			(effects
@@
 			)
 		)
-		(property "Footprint" ""
+		(property "Footprint" "Connector_PinHeader_2.54mm:PinHeader_1x02_P2.54mm_Vertical"
 			(at 603.25 129.54 0)
 			(effects
@@
 			)
 		)
-		(property "Footprint" ""
+		(property "Footprint" "Connector_RJ:RJ45_OST_PJ012-8P8CX_Vertical"
 			(at 774.7 182.245 90)
 			(effects
@@
 			)
 		)
-		(property "Footprint" ""
+		(property "Footprint" "Connector_RJ:RJ45_OST_PJ012-8P8CX_Vertical"
 			(at 703.58 182.245 90)
 			(effects
@@
 			)
 		)
-		(property "Footprint" ""
+		(property "Footprint" "TestPoint:TestPoint_Pad_D2.0mm"
 			(at 448.31 179.07 0)
 			(effects
@@
 			)
 		)
-		(property "Footprint" "Capacitors_SMD:C_0603"
+		(property "Footprint" "Capacitor_SMD:C_0603_1608Metric"
 			(at 244.8052 38.1 0)
 			(effects
@@
 			)
 		)
-		(property "Footprint" ""
+		(property "Footprint" "TestPoint:TestPoint_Pad_D2.0mm"
 			(at 448.31 171.45 0)
 			(effects
@@
 			)
 		)
-		(property "Footprint" ""
+		(property "Footprint" "TestPoint:TestPoint_Pad_D2.0mm"
 			(at 448.31 181.61 0)
 			(effects
@@
 			)
 		)
-		(property "Footprint" "Resistors_SMD:R_0603"
+		(property "Footprint" "Capacitor_SMD:C_0603_1608Metric"
 			(at 551.942 124.46 90)
 			(effects
@@
 			)
 		)
-		(property "Value" "~"
+		(property "Value" "MCP111"
 			(at 553.72 213.36 0)
 			(effects

Commit message: Assigning URLs.
Parts:
- D1, U10: URL (none) -> https://www.digikey.com/en/products/detail/stmicroelectroni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
- J6: URL (none) -> https://www.digikey.com/en/products/detail/on-shore-technol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
- L1: footprint (none) -> Inductor_SMD:L_1008_2520Metric; URL (none) -> https://www.digikey.com/en/products/detail/murata-electroni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
- U11, U12, U8, U9: URL (none) -> https://www.digikey.com/en/products/detail/microchip-techno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
- Y1: URL (none) -> https://www.digikey.com/en/products/detail/yic/8M20P2-49US/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
Changed lines of the file:
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@@
 			)
 		)
+		(property "URL" "https://www.digikey.com/en/products/detail/on-shore-technology-inc/USB-B1HSB6/2677744"
+			(at 168.91 353.06 0)
+			(effects
+				(font
+					(size 1.27 1.27)
+				)
+				(hide yes)
+			)
+		)
 		(pin "5"
 		)
@@
 			)
 		)
+		(property "URL" "https://www.digikey.com/en/products/detail/microchip-technology/MCP1603T-330I-OS/1098431"
+			(at 414.02 34.29 0)
+			(effects
+				(font
+					(size 1.27 1.27)
+				)
+				(hide yes)
+			)
+		)
 		(pin "5"
 		)
@@
 			)
 		)
+		(property "URL" "https://www.digikey.com/en/products/detail/stmicroelectronics/stm32f405rgt6/2754208"
+			(at 323.85 367.03 0)
+			(effects
+				(font
+					(size 1.27 1.27)
+				)
+				(hide yes)
+			)
+		)
 		(pin "11"
 		)
@@
 			)
 		)
+		(property "URL" "https://www.digikey.com/en/products/detail/stmicroelectronics/1N5819/1037326"
+			(at 269.24 49.53 90)
+			(effects
+				(font
+					(size 1.27 1.27)
+				)
+				(hide yes)
+			)
+		)
 		(pin "2"
 		)
@@
 			)
 		)
+		(property "URL" "https://www.digikey.com/en/products/detail/yic/8M20P2-49US/15648614"
+			(at 434.34 419.1 0)
+			(effects
+				(font
+					(size 1.27 1.27)
+				)
+				(hide yes)
+			)
+		)
 		(pin "2"
 		)
@@
 			)
 		)
+		(property "URL" "https://www.digikey.com/en/products/detail/stmicroelectronics/stm32f405rgt6/2754208"
+			(at 73.66 384.81 0)
+			(effects
+				(font
+					(size 1.27 1.27)
+				)
+				(hide yes)
+			)
+		)
 		(pin "11"
 		)
@@
 			)
 		)
+		(property "URL" "https://www.digikey.com/en/products/detail/microchip-technology/MCP73812T-420I-OT/1626618?s=N4IgTCBcDaILYGMAOB2AzADgIxgC4gF0BfIA"
+			(at 234.95 58.42 0)
+			(effects
+				(font
+					(size 1.27 1.27)
+				)
+				(hide yes)
+			)
+		)
 		(pin "4"
 		)
@@
 			)
 		)
-		(property "Footprint" ""
+		(property "Footprint" "Inductor_SMD:L_1008_2520Metric"
 			(at 431.8 29.21 0)
 			(effects
@@
 			)
 		)
-		(property "Description" "Inductor"
+		(property "Description" "LQM2HPN4R7MG0L"
 			(at 431.8 29.21 0)
 			(effects
@@
 			)
 		)
+		(property "URL" "https://www.digikey.com/en/products/detail/murata-electronics/LQM2HPN4R7MG0L/1893673"
+			(at 431.8 29.21 90)
+			(effects
+				(font
+					(size 1.27 1.27)
+				)
+				(hide yes)
+			)
+		)
 		(pin "2"
 		)
@@
 			)
 		)
+		(property "URL" "https://www.digikey.com/en/products/detail/microchip-technology/BM71BLES1FC2-0B02AA/7164757?s=N4IgTCBcDaIEIFkDsBGOAZAogZRQMQGEwBaABjlLAEEqQBdAXyA"
+			(at 421.64 123.19 0)
+			(effects
+				(font
+					(size 1.27 1.27)
+				)
+				(hide yes)
+			)
+		)
 		(pin "8"
 		)
@@
 			(at 560.07 212.09 0)
 			(effects
+				(font
+					(size 1.27 1.27)
+				)
+				(hide yes)
+			)
+		)
+		(property "URL" "https://www.digikey.com/en/products/detail/microchip-technology/MCP111T-315E-TT/716028"
+			(at 560.07 212.09 0)
+			(effects

Commit message: Assigning URLs...
Parts:
- C21, C22, C3, C32, C33, C34, C35, C6, C7, C8: URL (none) -> https://www.digikey.com/product-detail/en/samsung-electro-m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; url https://www.digikey.com/product-detail/en/samsung-electro-m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 -> (none)
- D2: URL (none) -> https://www.digikey.com/en/products/detail/stmicroelectroni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
- R83, R84, R85: URL (none) -> https://www.digikey.com/en/products/detail/yageo/AC0603JR-0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; url https://www.digikey.com/product-detail/en/yageo/RC0603JR-07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 -> (none)
- R86, R97: value 10k -> 10k 5%; URL (none) -> https://www.digikey.com/product-detail/en/yageo/RC0603JR-07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; url https://www.digikey.com/product-detail/en/yageo/RC0603JR-07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 -> (none)
- R87, R88, R89, R90, R92, R93, R98: URL (none) -> https://www.digikey.com/en/products/detail/yageo/RC0603JR-1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
- R91: URL (none) -> https://www.digikey.com/en/products/detail/yageo/AC0603JR-0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
- R96: URL (none) -> https://www.digikey.com/product-detail/en/yageo/RC0603JR-07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; url https://www.digikey.com/product-detail/en/yageo/RC0603JR-07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 -> (none)
Changed lines of the file:
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@@
 			)
 		)
-		(property "Value" "10k"
-			(at 590.55 172.72 90)
+		(property "Value" "10k 5%"
+			(at 588.01 172.72 90)
 			(effects
 				(font
@@
 			)
 		)
-		(property "url" "https://www.digikey.com/product-detail/en/yageo/RC0603JR-072K2L/311-2.2KGRCT-ND/729676"
+		(property "URL" "https://www.digikey.com/product-detail/en/yageo/RC0603JR-072K2L/311-2.2KGRCT-ND/729676"
 			(at 590.55 172.72 90)
 			(effects
@@
 			)
 		)
-		(property "url" "https://www.digikey.com/product-detail/en/samsung-electro-mechanics-america-inc/CL10B475KQ8NQNC/1276-2087-1-ND/3890173"
+		(property "URL" "https://www.digikey.com/product-detail/en/samsung-electro-mechanics-america-inc/CL10B475KQ8NQNC/1276-2087-1-ND/3890173"
 			(at 511.81 128.27 0)
 			(effects
@@
 			)
 		)
+		(property "URL" "https://www.digikey.com/en/products/detail/stmicroelectronics/1N5819/1037326"
+			(at 180.34 60.96 0)
+			(effects
+				(font
+					(size 1.27 1.27)
+				)
+				(hide yes)
+			)
+		)
 		(pin "2"
 		)
@@
 			)
 		)
+		(property "URL" "https://www.digikey.com/en/products/detail/yageo/RC0603JR-1010KL/13694233"
+			(at 424.18 317.5 90)
+			(effects
+				(font
+					(size 1.27 1.27)
+				)
+				(hide yes)
+			)
+		)
 		(pin "2"
 		)
@@
 			)
 		)
-		(property "url" "https://www.digikey.com/product-detail/en/yageo/RC0603JR-072K2L/311-2.2KGRCT-ND/729676"
+		(property "URL" "https://www.digikey.com/product-detail/en/yageo/RC0603JR-072K2L/311-2.2KGRCT-ND/729676"
 			(at 387.35 130.81 90)
 			(effects
@@
 			)
 		)
-		(property "url" "https://www.digikey.com/product-detail/en/samsung-electro-mechanics-america-inc/CL10B475KQ8NQNC/1276-2087-1-ND/3890173"
+		(property "URL" "https://www.digikey.com/product-detail/en/samsung-electro-mechanics-america-inc/CL10B475KQ8NQNC/1276-2087-1-ND/3890173"
 			(at 519.43 128.27 0)
 			(effects
@@
 			)
 		)
-		(property "url" "https://www.digikey.com/product-detail/en/yageo/RC0603JR-072K2L/311-2.2KGRCT-ND/729676"
+		(property "URL" "https://www.digikey.com/en/products/detail/yageo/AC0603JR-072K2L/5896418"
 			(at 213.36 77.47 90)
 			(effects
@@
 			)
 		)
-		(property "url" "https://www.digikey.com/product-detail/en/samsung-electro-mechanics-america-inc/CL10B475KQ8NQNC/1276-2087-1-ND/3890173"
+		(property "URL" "https://www.digikey.com/product-detail/en/samsung-electro-mechanics-america-inc/CL10B475KQ8NQNC/1276-2087-1-ND/3890173"
 			(at 247.65 62.23 0)
 			(effects
@@
 			)
 		)
-		(property "url" "https://www.digikey.com/product-detail/en/samsung-electro-mechanics-america-inc/CL10B475KQ8NQNC/1276-2087-1-ND/3890173"
+		(property "URL" "https://www.digikey.com/product-detail/en/samsung-electro-mechanics-america-inc/CL10B475KQ8NQNC/1276-2087-1-ND/3890173"
 			(at 527.05 128.27 0)
 			(effects
@@
 		)
 		(property "Value" "1k 5%"
-			(at 163.83 391.16 90)
+			(at 162.052 391.16 90)
 			(effects
 				(font
@@
 			)
 		)
+		(property "URL" "https://www.digikey.com/en/products/detail/yageo/RC0603JR-131KL/13694162"
+			(at 163.83 391.16 90)
+			(effects
+				(font
+					(size 1.27 1.27)
+				)
+				(hide yes)
+			)
+		)
 		(pin "1"
 		)
@@
 			)
 		)
-		(property "url" "https://www.digikey.com/product-detail/en/samsung-electro-mechanics-america-inc/CL10B475KQ8NQNC/1276-2087-1-ND/3890173"
+		(property "URL" "https://www.digikey.com/product-detail/en/samsung-electro-mechanics-america-inc/CL10B475KQ8NQNC/1276-2087-1-ND/3890173"
 			(at 449.58 35.56 0)
 			(effects
@@
 		)
 		(property "Value" "1k 5%"
-			(at 189.23 391.16 90)
+			(at 187.198 391.16 90)
 			(effects
 				(font
@@
 			)
 		)
+		(property "URL" "https://www.digikey.com/en/products/detail/yageo/RC0603JR-131KL/13694162"
+			(at 189.23 391.16 90)
+			(effects
+				(font
+					(size 1.27 1.27)
+				)
+				(hide yes)
+			)
+		)
 		(pin "1"
 		)
@@
 			)
 		)
-		(property "url" "https://www.digikey.com/product-detail/en/samsung-electro-mechanics-america-inc/CL10B475KQ8NQNC/1276-2087-1-ND/3890173"
+		(property "URL" "https://www.digikey.com/product-detail/en/samsung-electro-mechanics-america-inc/CL10B475KQ8NQNC/1276-2087-1-ND/3890173"
 			(at 590.55 189.23 0)
 			(effects
@@
 		)
 		(property "Value" "1k 5%"
-			(at 516.89 165.1 90)
+			(at 514.858 165.1 90)
 			(effects
 				(font
@@
 			)
 		)
+		(property "URL" "https://www.digikey.com/en/products/detail/yageo/RC0603JR-131KL/13694162"
+			(at 516.89 165.1 90)
+			(effects
+				(font
+					(size 1.27 1.27)
+				)
+				(hide yes)
+			)
+		)
 		(pin "1"
 		)
@@
 			)
 		)
-		(property "url" "https://www.digikey.com/product-detail/en/samsung-electro-mechanics-america-inc/CL10B475KQ8NQNC/1276-2087-1-ND/3890173"
+		(property "URL" "https://www.digikey.com/product-detail/en/samsung-electro-mechanics-america-inc/CL10B475KQ8NQNC/1276-2087-1-ND/3890173"
 			(at 553.72 140.97 0)
 			(effects
@@
 			)
 		)
-		(property "url" "https://www.digikey.com/product-detail/en/samsung-electro-mechanics-america-inc/CL10B475KQ8NQNC/1276-2087-1-ND/3890173"
+		(property "URL" "https://www.digikey.com/product-detail/en/samsung-electro-mechanics-america-inc/CL10B475KQ8NQNC/1276-2087-1-ND/3890173"
 			(at 381 35.56 0)
 			(effects
@@
 			)
 		)
-		(property "url" "https://www.digikey.com/product-detail/en/yageo/RC0603JR-072K2L/311-2.2KGRCT-ND/729676"
+		(property "URL" "https://www.digikey.com/en/products/detail/yageo/AC0603JR-072K2L/5896418"
 			(at 213.36 67.31 90)
 			(effects
@@
 			)
 		)
-		(property "url" "https://www.digikey.com/product-detail/en/yageo/RC0603JR-072K2L/311-2.2KGRCT-ND/729676"
+		(property "URL" "https://www.digikey.com/en/products/detail/yageo/AC0603JR-072K2L/5896418"
 			(at 213.36 87.63 90)
 			(effects
@@
 			)
 		)
+		(property "URL" "https://www.digikey.com/en/products/detail/yageo/RC0603JR-1010KL/13694233"
+			(at 179.07 304.8 90)
+			(effects
+				(font
+					(size 1.27 1.27)
+				)
+				(hide yes)
+			)
+		)
 		(pin "2"
 		)
@@
 			)
 		)
-		(property "url" "https://www.digikey.com/product-detail/en/samsung-electro-mechanics-america-inc/CL10B475KQ8NQNC/1276-2087-1-ND/3890173"
+		(property "URL" "https://www.digikey.com/product-detail/en/samsung-electro-mechanics-america-inc/CL10B475KQ8NQNC/1276-2087-1-ND/3890173"
 			(at 217.17 317.5 0)
 			(effects
@@
 		)
 		(property "Value" "10k 5%"
-			(at 424.18 373.38 90)
+			(at 426.974 373.634 90)
 			(effects
 				(font
@@
 			)
 		)
+		(property "URL" "https://www.digikey.com/en/products/detail/yageo/RC0603JR-1010KL/13694233"
+			(at 424.18 373.38 90)
+			(effects
+				(font
+					(size 1.27 1.27)
+				)
+				(hide yes)
+			)
+		)
 		(pin "1"
 		)
@@
 			)
 		)
-		(property "url" "https://www.digikey.com/product-detail/en/samsung-electro-mechanics-america-inc/CL10B475KQ8NQNC/1276-2087-1-ND/3890173"
+		(property "URL" "https://www.digikey.com/product-detail/en/samsung-electro-mechanics-america-inc/CL10B475KQ8NQNC/1276-2087-1-ND/3890173"
 			(at 243.84 34.29 0)
 			(effects
@@
 		)
 		(property "Value" "1k 5%"
-			(at 176.53 391.16 90)
+			(at 174.752 391.16 90)
 			(effects
 				(font
@@
 			)
 		)
+		(property "URL" "https://www.digikey.com/en/products/detail/yageo/RC0603JR-131KL/13694162"
+			(at 176.53 391.16 90)
+			(effects
+				(font
+					(size 1.27 1.27)
+				)
+				(hide yes)
+			)
+		)
 		(pin "1"
 		)
@@
 			)
 		)
-		(property "Value" "10k"
-			(at 553.72 124.46 90)
+		(property "Value" "10k 5%"
+			(at 551.434 124.46 90)
 			(effects
 				(font
@@
 			)
 		)
-		(property "url" "https://www.digikey.com/product-detail/en/yageo/RC0603JR-072K2L/311-2.2KGRCT-ND/729676"
+		(property "URL" "https://www.digikey.com/product-detail/en/yageo/RC0603JR-072K2L/311-2.2KGRCT-ND/729676"
 			(at 553.72 124.46 90)
 			(effects
@@
 			(effects
 				(font
+					(size 1.27 1.27)
+				)
+				(hide yes)
+			)
+		)
+		(property "URL" "https://www.digikey.com/en/products/detail/yageo/AC0603JR-07100RL/5896356"
+			(at 450.85 422.91 90)
+			(effects
+				(font
