File: schematics/multi_sensor_host/parallel_input.kicad_sch (KiCad schematic)
At the start: 14 parts, among them U4 74HC165

Commit message: Cannot re-save stm32f405rgt6. May be need to copy it again from the other project.
Parts:
- C25, C26: symbol multi_i2c-rescue:C -> Device:C
- R50, R51, R52, R53, R54, R55, R56, R57, R58, R59, R60: symbol multi_i2c-rescue:R -> Device:R
Changed lines of the file:
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@@
 	)
 	(symbol
-		(lib_id "multi_i2c-rescue:R")
+		(lib_id "Device:R")
 		(at 118.11 90.17 90)
 		(unit 1)
@@
 			)
 		)
-		(property "Datasheet" ""
+		(property "Datasheet" "~"
 			(at 118.11 90.17 0)
 			(effects
@@
 			)
 		)
-		(property "Description" "RC0603JR-072K2L"
-			(at 118.11 90.17 90)
-			(effects
-				(font
-					(size 1.524 1.524)
+		(property "Description" "Resistor"
+			(at 118.11 90.17 0)
+			(effects
+				(font
+					(size 1.27 1.27)
 				)
 				(hide yes)
@@
 	)
 	(symbol
-		(lib_id "multi_i2c-rescue:R")
+		(lib_id "Device:R")
 		(at 118.11 97.79 90)
 		(unit 1)
@@
 			)
 		)
-		(property "Datasheet" ""
+		(property "Datasheet" "~"
 			(at 118.11 97.79 0)
 			(effects
@@
 			)
 		)
-		(property "Description" "RC0603JR-072K2L"
-			(at 118.11 97.79 90)
-			(effects
-				(font
-					(size 1.524 1.524)
+		(property "Description" "Resistor"
+			(at 118.11 97.79 0)
+			(effects
+				(font
+					(size 1.27 1.27)
 				)
 				(hide yes)
@@
 	)
 	(symbol
-		(lib_id "multi_i2c-rescue:R")
+		(lib_id "Device:R")
 		(at 118.11 102.87 90)
 		(unit 1)
@@
 			)
 		)
-		(property "Datasheet" ""
+		(property "Datasheet" "~"
 			(at 118.11 102.87 0)
 			(effects
@@
 			)
 		)
-		(property "Description" "RC0603JR-072K2L"
-			(at 118.11 102.87 90)
-			(effects
-				(font
-					(size 1.524 1.524)
+		(property "Description" "Resistor"
+			(at 118.11 102.87 0)
+			(effects
+				(font
+					(size 1.27 1.27)
 				)
 				(hide yes)
@@
 	)
 	(symbol
-		(lib_id "multi_i2c-rescue:C")
+		(lib_id "Device:C")
 		(at 168.91 63.5 0)
 		(unit 1)
@@
 			)
 		)
-		(property "Datasheet" ""
+		(property "Datasheet" "~"
 			(at 168.91 63.5 0)
 			(effects
@@
 			)
 		)
-		(property "Description" "CC0603KRX7R7BB104"
+		(property "Description" "Unpolarized capacitor"
 			(at 168.91 63.5 0)
 			(effects
 				(font
-					(size 1.524 1.524)
+					(size 1.27 1.27)
 				)
 				(hide yes)
@@
 	)
 	(symbol
-		(lib_id "multi_i2c-rescue:GND")
+		(lib_id "power:GND")
 		(at 134.62 118.11 0)
 		(unit 1)
@@
 			)
 		)
-		(property "Description" ""
+		(property "Description" "Power symbol creates a global label with name \"GND\" , ground"
 			(at 134.62 118.11 0)
 			(effects
@@
 	)
 	(symbol
-		(lib_id "multi_i2c-rescue:GND")
+		(lib_id "power:GND")
 		(at 168.91 69.85 0)
 		(unit 1)
@@
 			)
 		)
-		(property "Description" ""
+		(property "Description" "Power symbol creates a global label with name \"GND\" , ground"
 			(at 168.91 69.85 0)
 			(effects
@@
 	)
 	(symbol
-		(lib_id "multi_i2c-rescue:R")
+		(lib_id "Device:R")
 		(at 118.11 113.03 90)
 		(unit 1)
@@
 			)
 		)
-		(property "Datasheet" ""
+		(property "Datasheet" "~"
 			(at 118.11 113.03 0)
 			(effects
@@
 			)
 		)
-		(property "Description" "RC0603JR-072K2L"
-			(at 118.11 113.03 90)
-			(effects
-				(font
-					(size 1.524 1.524)
+		(property "Description" "Resistor"
+			(at 118.11 113.03 0)
+			(effects
+				(font
+					(size 1.27 1.27)
 				)
 				(hide yes)
@@
 	)
 	(symbol
-		(lib_id "multi_i2c-rescue:R")
+		(lib_id "Device:R")
 		(at 193.04 82.55 90)
 		(unit 1)
@@
 			)
 		)
-		(property "Datasheet" ""
+		(property "Datasheet" "~"
 			(at 193.04 82.55 0)
 			(effects
@@
 			)
 		)
-		(property "Description" "RC0603JR-072K2L"
-			(at 193.04 82.55 90)
-			(effects
-				(font
-					(size 1.524 1.524)
+		(property "Description" "Resistor"
+			(at 193.04 82.55 0)
+			(effects
+				(font
+					(size 1.27 1.27)
 				)
 				(hide yes)
@@
 	)
 	(symbol
-		(lib_id "multi_i2c-rescue:R")
+		(lib_id "Device:R")
 		(at 118.11 95.25 90)
 		(unit 1)
@@
 			)
 		)
-		(property "Datasheet" ""
+		(property "Datasheet" "~"
 			(at 118.11 95.25 0)
 			(effects
@@
 			)
 		)
-		(property "Description" "RC0603JR-072K2L"
-			(at 118.11 95.25 90)
-			(effects
-				(font
-					(size 1.524 1.524)
+		(property "Description" "Resistor"
+			(at 118.11 95.25 0)
+			(effects
+				(font
+					(size 1.27 1.27)
 				)
 				(hide yes)
@@
 	)
 	(symbol
-		(lib_id "multi_i2c-rescue:R")
+		(lib_id "Device:R")
 		(at 118.11 85.09 90)
 		(unit 1)
@@
 			)
 		)
-		(property "Datasheet" ""
+		(property "Datasheet" "~"
 			(at 118.11 85.09 0)
 			(effects
@@
 			)
 		)
-		(property "Description" "RC0603JR-072K2L"
-			(at 118.11 85.09 90)
-			(effects
-				(font
-					(size 1.524 1.524)
+		(property "Description" "Resistor"
+			(at 118.11 85.09 0)
+			(effects
+				(font
+					(size 1.27 1.27)
 				)
 				(hide yes)
@@
 	)
 	(symbol
-		(lib_id "multi_i2c-rescue:GND")
+		(lib_id "power:GND")
 		(at 177.8 69.85 0)
 		(unit 1)
@@
 			)
 		)
-		(property "Description" ""
+		(property "Description" "Power symbol creates a global label with name \"GND\" , ground"
 			(at 177.8 69.85 0)
 			(effects
@@
 	)
 	(symbol
-		(lib_id "multi_i2c-rescue:R")
+		(lib_id "Device:R")
 		(at 118.11 100.33 90)
 		(unit 1)
@@
 			)
 		)
-		(property "Datasheet" ""
+		(property "Datasheet" "~"
 			(at 118.11 100.33 0)
 			(effects
@@
 			)
 		)
-		(property "Description" "RC0603JR-072K2L"
-			(at 118.11 100.33 90)
-			(effects
-				(font
-					(size 1.524 1.524)
+		(property "Description" "Resistor"
+			(at 118.11 100.33 0)
+			(effects
+				(font
+					(size 1.27 1.27)
 				)
 				(hide yes)
@@
 	)
 	(symbol
-		(lib_id "multi_i2c-rescue:R")
+		(lib_id "Device:R")
 		(at 118.11 92.71 90)
 		(unit 1)
@@
 			)
 		)
-		(property "Datasheet" ""
+		(property "Datasheet" "~"
 			(at 118.11 92.71 0)
 			(effects
@@
 			)
 		)
-		(property "Description" "RC0603JR-072K2L"
-			(at 118.11 92.71 90)
-			(effects
-				(font
-					(size 1.524 1.524)
+		(property "Description" "Resistor"
+			(at 118.11 92.71 0)
+			(effects
+				(font
+					(size 1.27 1.27)
 				)
 				(hide yes)
@@
 	)
 	(symbol
-		(lib_id "multi_i2c-rescue:C")
+		(lib_id "Device:C")
 		(at 177.8 63.5 0)
 		(unit 1)
@@
 			)
 		)
-		(property "Datasheet" ""
+		(property "Datasheet" "~"
 			(at 177.8 63.5 0)
 			(effects
@@
 			)
 		)
-		(property "Description" "CL10B475KQ8NQNC"
+		(property "Description" "Unpolarized capacitor"
 			(at 177.8 63.5 0)
 			(effects
 				(font
-					(size 1.524 1.524)
+					(size 1.27 1.27)
 				)
 				(hide yes)
@@
 	)
 	(symbol
-		(lib_id "multi_i2c-rescue:GND")
+		(lib_id "power:GND")
 		(at 149.86 128.27 0)
 		(unit 1)
@@
 			)
 		)
-		(property "Description" ""
+		(property "Description" "Power symbol creates a global label with name \"GND\" , ground"
 			(at 149.86 128.27 0)
 			(effects
@@
 	)
 	(symbol
-		(lib_id "multi_i2c-rescue:R")
+		(lib_id "Device:R")
 		(at 118.11 107.95 90)
 		(unit 1)
@@
 			)
 		)
-		(property "Datasheet" ""
+		(property "Datasheet" "~"
 			(at 118.11 107.95 0)
 			(effects
@@
 			)
 		)
-		(property "Description" "RC0603JR-072K2L"
-			(at 118.11 107.95 90)
-			(effects
-				(font
-					(size 1.524 1.524)
+		(property "Description" "Resistor"
+			(at 118.11 107.95 0)
+			(effects
+				(font
+					(size 1.27 1.27)
 				)
 				(hide yes)
@@
 	)
 	(symbol
-		(lib_id "multi_i2c-rescue:R")
+		(lib_id "Device:R")
 		(at 118.11 87.63 90)
 		(unit 1)
@@
 			)
 		)
-		(property "Datasheet" ""
+		(property "Datasheet" "~"
 			(at 118.11 87.63 0)
 			(effects
@@
 			)
 		)
-		(property "Description" "RC0603JR-072K2L"
-			(at 118.11 87.63 90)
-			(effects
-				(font
-					(size 1.524 1.524)
-				)
-				(hide yes)
+		(property "Description" "Resistor"
+			(at 118.11 87.63 0)
+			(effects
+				(font
+					(size 1.27 1.27)
+				)
+				(hide yes)

Commit message: No errors, no warnings.
Changed lines of the file:
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@@
 	)
 	(symbol
-		(lib_id "multi_i2c-rescue:VDD")
+		(lib_id "power:VDD")
 		(at 149.86 54.61 0)
 		(unit 1)
@@
 			)
 		)
-		(property "Description" ""
+		(property "Description" "Power symbol creates a global label with name \"VDD\""
 			(at 149.86 54.61 0)
 			(effects

Commit message: Assigned footprints. Also, just in case found a chip I2C to diff. pair.
Parts:
- C25, C26: footprint Capacitors_SMD:C_0603 -> Capacitor_SMD:C_0603_1608Metric
- R50, R51, R52, R53, R54, R55, R56, R57, R58, R59, R60: footprint Resistors_SMD:R_0603 -> Capacitor_SMD:C_0603_1608Metric
- U4: footprint (none) -> Package_SO:SO-16_3.9x9.9mm_P1.27mm
Changed lines of the file:
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@@
 			)
 		)
-		(property "Footprint" "Resistors_SMD:R_0603"
+		(property "Footprint" "Capacitor_SMD:C_0603_1608Metric"
 			(at 118.11 91.948 90)
 			(effects
@@
 			)
 		)
-		(property "Footprint" "Resistors_SMD:R_0603"
+		(property "Footprint" "Capacitor_SMD:C_0603_1608Metric"
 			(at 118.11 99.568 90)
 			(effects
@@
 			)
 		)
-		(property "Footprint" "Resistors_SMD:R_0603"
+		(property "Footprint" "Capacitor_SMD:C_0603_1608Metric"
 			(at 118.11 104.648 90)
 			(effects
@@
 			)
 		)
-		(property "Footprint" "Capacitors_SMD:C_0603"
+		(property "Footprint" "Capacitor_SMD:C_0603_1608Metric"
 			(at 169.8752 67.31 0)
 			(effects
@@
 			)
 		)
-		(property "Footprint" "Resistors_SMD:R_0603"
+		(property "Footprint" "Capacitor_SMD:C_0603_1608Metric"
 			(at 118.11 114.808 90)
 			(effects
@@
 			)
 		)
-		(property "Footprint" ""
+		(property "Footprint" "Package_SO:SO-16_3.9x9.9mm_P1.27mm"
 			(at 149.86 97.79 0)
 			(effects
@@
 			)
 		)
-		(property "Footprint" "Resistors_SMD:R_0603"
+		(property "Footprint" "Capacitor_SMD:C_0603_1608Metric"
 			(at 193.04 84.328 90)
 			(effects
@@
 			)
 		)
-		(property "Footprint" "Resistors_SMD:R_0603"
+		(property "Footprint" "Capacitor_SMD:C_0603_1608Metric"
 			(at 118.11 97.028 90)
 			(effects
@@
 			)
 		)
-		(property "Footprint" "Resistors_SMD:R_0603"
+		(property "Footprint" "Capacitor_SMD:C_0603_1608Metric"
 			(at 118.11 86.868 90)
 			(effects
@@
 			)
 		)
-		(property "Footprint" "Resistors_SMD:R_0603"
+		(property "Footprint" "Capacitor_SMD:C_0603_1608Metric"
 			(at 118.11 102.108 90)
 			(effects
@@
 			)
 		)
-		(property "Footprint" "Resistors_SMD:R_0603"
+		(property "Footprint" "Capacitor_SMD:C_0603_1608Metric"
 			(at 118.11 94.488 90)
 			(effects
@@
 			)
 		)
-		(property "Footprint" "Capacitors_SMD:C_0603"
+		(property "Footprint" "Capacitor_SMD:C_0603_1608Metric"
 			(at 178.7652 67.31 0)
 			(effects
@@
 			)
 		)
-		(property "Footprint" "Resistors_SMD:R_0603"
+		(property "Footprint" "Capacitor_SMD:C_0603_1608Metric"
 			(at 118.11 109.728 90)
 			(effects
@@
 			)
 		)
-		(property "Footprint" "Resistors_SMD:R_0603"
+		(property "Footprint" "Capacitor_SMD:C_0603_1608Metric"
 			(at 118.11 89.408 90)
 			(effects

Commit message: Assigning URLs.
Parts:
- U4: URL (none) -> https://www.digikey.com/en/products/detail/nexperia-usa-inc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
Changed lines of the file:
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@@
+			)
+		)
+		(property "URL" "https://www.digikey.com/en/products/detail/nexperia-usa-inc/74LV165D-118/1231120"
+			(at 149.86 97.79 0)
+			(effects
+				(font
+					(size 1.27 1.27)
+				)
+				(hide yes)
 			)
 		)

Commit message: Assigning URLs...
Parts:
- C25: URL (none) -> https://www.digikey.com/product-detail/en/yageo/CC0603KRX7R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; url https://www.digikey.com/product-detail/en/yageo/CC0603KRX7R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 -> (none)
- C26: URL (none) -> https://www.digikey.com/product-detail/en/samsung-electro-m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; url https://www.digikey.com/product-detail/en/samsung-electro-m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 -> (none)
- R50, R51, R52, R53, R54, R55, R56, R57, R58, R59, R60: URL (none) -> https://www.digikey.com/en/products/detail/yageo/AC0603JR-0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; url https://www.digikey.com/product-detail/en/yageo/RC0603JR-07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 -> (none)
Changed lines of the file:
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@@
 			)
 		)
-		(property "url" "https://www.digikey.com/product-detail/en/yageo/RC0603JR-072K2L/311-2.2KGRCT-ND/729676"
+		(property "URL" "https://www.digikey.com/en/products/detail/yageo/AC0603JR-072K2L/5896418"
 			(at 118.11 90.17 90)
 			(effects
@@
 			)
 		)
-		(property "url" "https://www.digikey.com/product-detail/en/yageo/RC0603JR-072K2L/311-2.2KGRCT-ND/729676"
+		(property "URL" "https://www.digikey.com/en/products/detail/yageo/AC0603JR-072K2L/5896418"
 			(at 118.11 97.79 90)
 			(effects
@@
 			)
 		)
-		(property "url" "https://www.digikey.com/product-detail/en/yageo/RC0603JR-072K2L/311-2.2KGRCT-ND/729676"
+		(property "URL" "https://www.digikey.com/en/products/detail/yageo/AC0603JR-072K2L/5896418"
 			(at 118.11 102.87 90)
 			(effects
@@
 			)
 		)
-		(property "url" "https://www.digikey.com/product-detail/en/yageo/CC0603KRX7R7BB104/311-1088-1-ND/302998"
+		(property "URL" "https://www.digikey.com/product-detail/en/yageo/CC0603KRX7R7BB104/311-1088-1-ND/302998"
 			(at 168.91 63.5 0)
 			(effects
@@
 			)
 		)
-		(property "url" "https://www.digikey.com/product-detail/en/yageo/RC0603JR-072K2L/311-2.2KGRCT-ND/729676"
+		(property "URL" "https://www.digikey.com/en/products/detail/yageo/AC0603JR-072K2L/5896418"
 			(at 118.11 113.03 90)
 			(effects
@@
 			)
 		)
-		(property "url" "https://www.digikey.com/product-detail/en/yageo/RC0603JR-072K2L/311-2.2KGRCT-ND/729676"
+		(property "URL" "https://www.digikey.com/en/products/detail/yageo/AC0603JR-072K2L/5896418"
 			(at 193.04 82.55 90)
 			(effects
@@
 			)
 		)
-		(property "url" "https://www.digikey.com/product-detail/en/yageo/RC0603JR-072K2L/311-2.2KGRCT-ND/729676"
+		(property "URL" "https://www.digikey.com/en/products/detail/yageo/AC0603JR-072K2L/5896418"
 			(at 118.11 95.25 90)
 			(effects
@@
 			)
 		)
-		(property "url" "https://www.digikey.com/product-detail/en/yageo/RC0603JR-072K2L/311-2.2KGRCT-ND/729676"
+		(property "URL" "https://www.digikey.com/en/products/detail/yageo/AC0603JR-072K2L/5896418"
 			(at 118.11 85.09 90)
 			(effects
@@
 			)
 		)
-		(property "url" "https://www.digikey.com/product-detail/en/yageo/RC0603JR-072K2L/311-2.2KGRCT-ND/729676"
+		(property "URL" "https://www.digikey.com/en/products/detail/yageo/AC0603JR-072K2L/5896418"
 			(at 118.11 100.33 90)
 			(effects
@@
 			)
 		)
-		(property "url" "https://www.digikey.com/product-detail/en/yageo/RC0603JR-072K2L/311-2.2KGRCT-ND/729676"
+		(property "URL" "https://www.digikey.com/en/products/detail/yageo/AC0603JR-072K2L/5896418"
 			(at 118.11 92.71 90)
 			(effects
@@
 			)
 		)
-		(property "url" "https://www.digikey.com/product-detail/en/samsung-electro-mechanics-america-inc/CL10B475KQ8NQNC/1276-2087-1-ND/3890173"
+		(property "URL" "https://www.digikey.com/product-detail/en/samsung-electro-mechanics-america-inc/CL10B475KQ8NQNC/1276-2087-1-ND/3890173"
 			(at 177.8 63.5 0)
 			(effects
@@
 			)
 		)
-		(property "url" "https://www.digikey.com/product-detail/en/yageo/RC0603JR-072K2L/311-2.2KGRCT-ND/729676"
+		(property "URL" "https://www.digikey.com/en/products/detail/yageo/AC0603JR-072K2L/5896418"
 			(at 118.11 107.95 90)
 			(effects
@@
 			)
 		)
-		(property "url" "https://www.digikey.com/product-detail/en/yageo/RC0603JR-072K2L/311-2.2KGRCT-ND/729676"
+		(property "URL" "https://www.digikey.com/en/products/detail/yageo/AC0603JR-072K2L/5896418"
 			(at 118.11 87.63 90)
 			(effects

Commit message: Placing components...
Parts:
- R50, R51, R52, R53, R54, R55, R56, R57, R58, R59, R60: footprint Capacitor_SMD:C_0603_1608Metric -> Resistor_SMD:R_0603_1608Metric
Changed lines of the file:
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@@
-		)
-	)
-	(label "data_3"
-		(at 99.06 92.71 0)
-		(fields_autoplaced yes)
-		(effects
-			(font
-				(size 1.27 1.27)
-			)
-			(justify left bottom)
-		)
-	)
-	(label "serial_output"
-		(at 200.66 82.55 0)
-		(fields_autoplaced yes)
-		(effects
-			(font
-				(size 1.27 1.27)
-			)
-			(justify left bottom)
-		)
-	)
-	(label "parallel_load"
-		(at 99.06 107.95 0)
-		(fields_autoplaced yes)
-		(effects
-			(font
-				(size 1.27 1.27)
-			)
-			(justify left bottom)
-		)
-	)
-	(label "data_1"
-		(at 99.06 87.63 0)
-		(fields_autoplaced yes)
-		(effects
-			(font
-				(size 1.27 1.27)
-			)
-			(justify left bottom)
-		)
-	)
-	(label "data_serial"
-		(at 123.19 82.55 0)
-		(fields_autoplaced yes)
-		(effects
-			(font
-				(size 1.27 1.27)
-			)
-			(justify left bottom)
-		)
-	)
-	(label "data_0"
-		(at 99.06 85.09 0)
-		(fields_autoplaced yes)
-		(effects
-			(font
-				(size 1.27 1.27)
-			)
-			(justify left bottom)
-		)
-	)
-	(label "data_4"
-		(at 99.06 95.25 0)
-		(fields_autoplaced yes)
-		(effects
-			(font
-				(size 1.27 1.27)
-			)
-			(justify left bottom)
-		)
-	)
-	(label "data_2"
-		(at 99.06 90.17 0)
-		(fields_autoplaced yes)
-		(effects
-			(font
-				(size 1.27 1.27)
-			)
-			(justify left bottom)
-		)
-	)
-	(label "data_7"
-		(at 99.06 102.87 0)
-		(fields_autoplaced yes)
-		(effects
-			(font
-				(size 1.27 1.27)
-			)
-			(justify left bottom)
-		)
-	)
-	(label "data_5"
-		(at 99.06 97.79 0)
-		(fields_autoplaced yes)
-		(effects
-			(font
-				(size 1.27 1.27)
-			)
-			(justify left bottom)
-		)
-	)
-	(label "shifter_clock"
-		(at 99.06 113.03 0)
-		(fields_autoplaced yes)
-		(effects
-			(font
-				(size 1.27 1.27)
-			)
-			(justify left bottom)
-		)
-	)
-	(label "data_6"
-		(at 99.06 100.33 0)
-		(fields_autoplaced yes)
-		(effects
-			(font
-				(size 1.27 1.27)
-			)
-			(justify left bottom)
 		)
 	)
@@
 			)
 		)
-		(property "Footprint" "Capacitor_SMD:C_0603_1608Metric"
+		(property "Footprint" "Resistor_SMD:R_0603_1608Metric"
 			(at 118.11 91.948 90)
 			(effects
@@
 			)
 		)
-		(property "Footprint" "Capacitor_SMD:C_0603_1608Metric"
+		(property "Footprint" "Resistor_SMD:R_0603_1608Metric"
 			(at 118.11 99.568 90)
 			(effects
@@
 			)
 		)
-		(property "Footprint" "Capacitor_SMD:C_0603_1608Metric"
+		(property "Footprint" "Resistor_SMD:R_0603_1608Metric"
 			(at 118.11 104.648 90)
 			(effects
@@
 			)
 		)
-		(property "Footprint" "Capacitor_SMD:C_0603_1608Metric"
+		(property "Footprint" "Resistor_SMD:R_0603_1608Metric"
 			(at 118.11 114.808 90)
 			(effects
@@
 			)
 		)
-		(property "Footprint" "Capacitor_SMD:C_0603_1608Metric"
+		(property "Footprint" "Resistor_SMD:R_0603_1608Metric"
 			(at 193.04 84.328 90)
 			(effects
@@
 			)
 		)
-		(property "Footprint" "Capacitor_SMD:C_0603_1608Metric"
+		(property "Footprint" "Resistor_SMD:R_0603_1608Metric"
 			(at 118.11 97.028 90)
 			(effects
@@
 			)
 		)
-		(property "Footprint" "Capacitor_SMD:C_0603_1608Metric"
+		(property "Footprint" "Resistor_SMD:R_0603_1608Metric"
 			(at 118.11 86.868 90)
 			(effects
@@
 			)
 		)
-		(property "Footprint" "Capacitor_SMD:C_0603_1608Metric"
+		(property "Footprint" "Resistor_SMD:R_0603_1608Metric"
 			(at 118.11 102.108 90)
 			(effects
@@
 			)
 		)
-		(property "Footprint" "Capacitor_SMD:C_0603_1608Metric"
+		(property "Footprint" "Resistor_SMD:R_0603_1608Metric"
 			(at 118.11 94.488 90)
 			(effects
@@
 			)
 		)
-		(property "Footprint" "Capacitor_SMD:C_0603_1608Metric"
+		(property "Footprint" "Resistor_SMD:R_0603_1608Metric"
 			(at 118.11 109.728 90)
 			(effects
@@
 			)
 		)
-		(property "Footprint" "Capacitor_SMD:C_0603_1608Metric"
+		(property "Footprint" "Resistor_SMD:R_0603_1608Metric"
 			(at 118.11 89.408 90)
 			(effects
