File: schematics/multi_sensor_host/tca9548a_sheet.kicad_sch (KiCad schematic)
At the start: 23 parts, among them U1 TCA9548A_TSSOP

Commit message: Assigning URLs...
Parts:
- C1, C11: URL (none) -> https://www.digikey.com/product-detail/en/yageo/CC0603KRX7R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; url https://www.digikey.com/product-detail/en/yageo/CC0603KRX7R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 -> (none)
- C2: URL (none) -> https://www.digikey.com/product-detail/en/samsung-electro-m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; url https://www.digikey.com/product-detail/en/samsung-electro-m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 -> (none)
- R1: value 2k -> 10k 5%; URL (none) -> https://www.digikey.com/product-detail/en/yageo/RC0603JR-07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; url https://www.digikey.com/product-detail/en/yageo/RC0603JR-07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 -> (none)
- R10, R11, R12, R13, R14, R15, R16, R17, R18, R19, R2, R20, R21, R22, R23, R24, R25, R3: URL (none) -> https://www.digikey.com/en/products/detail/yageo/AC0603JR-0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; url https://www.digikey.com/product-detail/en/yageo/RC0603JR-07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 -> (none)
Changed lines of the file:
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@@
 			)
 		)
-		(property "url" "https://www.digikey.com/product-detail/en/yageo/RC0603JR-072K2L/311-2.2KGRCT-ND/729676"
+		(property "URL" "https://www.digikey.com/en/products/detail/yageo/AC0603JR-072K2L/5896418"
 			(at 213.36 68.58 90)
 			(effects
@@
 			)
 		)
-		(property "url" "https://www.digikey.com/product-detail/en/yageo/RC0603JR-072K2L/311-2.2KGRCT-ND/729676"
+		(property "URL" "https://www.digikey.com/en/products/detail/yageo/AC0603JR-072K2L/5896418"
 			(at 213.36 48.26 90)
 			(effects
@@
 			)
 		)
-		(property "url" "https://www.digikey.com/product-detail/en/yageo/RC0603JR-072K2L/311-2.2KGRCT-ND/729676"
+		(property "URL" "https://www.digikey.com/en/products/detail/yageo/AC0603JR-072K2L/5896418"
 			(at 213.36 129.54 90)
 			(effects
@@
 			)
 		)
-		(property "url" "https://www.digikey.com/product-detail/en/yageo/CC0603KRX7R7BB104/311-1088-1-ND/302998"
+		(property "URL" "https://www.digikey.com/product-detail/en/yageo/CC0603KRX7R7BB104/311-1088-1-ND/302998"
 			(at 95.25 139.7 0)
 			(effects
@@
 			)
 		)
-		(property "url" "https://www.digikey.com/product-detail/en/yageo/RC0603JR-072K2L/311-2.2KGRCT-ND/729676"
+		(property "URL" "https://www.digikey.com/en/products/detail/yageo/AC0603JR-072K2L/5896418"
 			(at 224.79 48.26 90)
 			(effects
@@
 	)
 	(symbol
-		(lib_id "Device:R")
-		(at 95.25 127 0)
-		(unit 1)
-		(exclude_from_sim no)
-		(in_bom yes)
-		(on_board yes)
-		(dnp no)
-		(property "Reference" "R1"
-			(at 97.282 127 90)
-			(effects
-				(font
-					(size 1.27 1.27)
-				)
-			)
-		)
-		(property "Value" "2k"
-			(at 95.25 127 90)
-			(effects
-				(font
-					(size 1.27 1.27)
-				)
-			)
-		)
-		(property "Footprint" "Capacitor_SMD:C_0603_1608Metric"
-			(at 93.472 127 90)
-			(effects
-				(font
-					(size 1.27 1.27)
-				)
-				(hide yes)
-			)
-		)
-		(property "Datasheet" "~"
-			(at 95.25 127 0)
-			(effects
-				(font
-					(size 1.27 1.27)
-				)
-				(hide yes)
-			)
-		)
-		(property "Description" "Resistor"
-			(at 95.25 127 0)
-			(effects
-				(font
-					(size 1.27 1.27)
-				)
-				(hide yes)
-			)
-		)
-		(property "url" "https://www.digikey.com/product-detail/en/yageo/RC0603JR-072K2L/311-2.2KGRCT-ND/729676"
-			(at 95.25 127 90)
-			(effects
-				(font
-					(size 1.524 1.524)
-				)
-				(hide yes)
-			)
-		)
-		(pin "2"
-		)
-		(pin "1"
-		)
-		(instances
-			(project "multi_sensor_host"
-				(path "/895fe915-d6d4-4da2-a6ec-6414a345dc15/46e9a6e6-b007-46d9-9be8-93a48bc459dd"
-					(reference "R1")
-					(unit 1)
-				)
-				(path "/895fe915-d6d4-4da2-a6ec-6414a345dc15/4b2528f7-9d95-4490-9078-a08d5cbf26f8"
-					(reference "R4")
-					(unit 1)
-				)
-			)
-		)
-	)
-	(symbol
 		(lib_id "Device:C")
 		(at 177.8 91.44 0)
@@
 			)
 		)
-		(property "url" "https://www.digikey.com/product-detail/en/yageo/CC0603KRX7R7BB104/311-1088-1-ND/302998"
+		(property "URL" "https://www.digikey.com/product-detail/en/yageo/CC0603KRX7R7BB104/311-1088-1-ND/302998"
 			(at 177.8 91.44 0)
 			(effects
@@
 			)
 		)
-		(property "url" "https://www.digikey.com/product-detail/en/yageo/RC0603JR-072K2L/311-2.2KGRCT-ND/729676"
+		(property "URL" "https://www.digikey.com/en/products/detail/yageo/AC0603JR-072K2L/5896418"
 			(at 224.79 109.22 90)
 			(effects
@@
 			)
 		)
-		(property "url" "https://www.digikey.com/product-detail/en/yageo/RC0603JR-072K2L/311-2.2KGRCT-ND/729676"
+		(property "URL" "https://www.digikey.com/en/products/detail/yageo/AC0603JR-072K2L/5896418"
 			(at 224.79 88.9 90)
 			(effects
@@
 			)
 		)
-		(property "url" "https://www.digikey.com/product-detail/en/yageo/RC0603JR-072K2L/311-2.2KGRCT-ND/729676"
+		(property "URL" "https://www.digikey.com/en/products/detail/yageo/AC0603JR-072K2L/5896418"
 			(at 143.51 114.3 90)
 			(effects
@@
 			)
 		)
-		(property "url" "https://www.digikey.com/product-detail/en/yageo/RC0603JR-072K2L/311-2.2KGRCT-ND/729676"
+		(property "URL" "https://www.digikey.com/en/products/detail/yageo/AC0603JR-072K2L/5896418"
 			(at 116.84 116.84 90)
 			(effects
@@
 			)
 		)
-		(property "url" "https://www.digikey.com/product-detail/en/yageo/RC0603JR-072K2L/311-2.2KGRCT-ND/729676"
+		(property "URL" "https://www.digikey.com/en/products/detail/yageo/AC0603JR-072K2L/5896418"
 			(at 213.36 109.22 90)
 			(effects
@@
 			)
 		)
-		(property "url" "https://www.digikey.com/product-detail/en/yageo/RC0603JR-072K2L/311-2.2KGRCT-ND/729676"
+		(property "URL" "https://www.digikey.com/en/products/detail/yageo/AC0603JR-072K2L/5896418"
 			(at 213.36 149.86 90)
 			(effects
@@
 			)
 		)
-		(property "url" "https://www.digikey.com/product-detail/en/yageo/RC0603JR-072K2L/311-2.2KGRCT-ND/729676"
+		(property "URL" "https://www.digikey.com/en/products/detail/yageo/AC0603JR-072K2L/5896418"
 			(at 213.36 190.5 90)
 			(effects
@@
 			)
 		)
-		(property "url" "https://www.digikey.com/product-detail/en/yageo/RC0603JR-072K2L/311-2.2KGRCT-ND/729676"
+		(property "URL" "https://www.digikey.com/en/products/detail/yageo/AC0603JR-072K2L/5896418"
 			(at 224.79 129.54 90)
 			(effects
@@
 			)
 		)
-		(property "url" "https://www.digikey.com/product-detail/en/yageo/RC0603JR-072K2L/311-2.2KGRCT-ND/729676"
+		(property "URL" "https://www.digikey.com/en/products/detail/yageo/AC0603JR-072K2L/5896418"
 			(at 224.79 68.58 90)
 			(effects
@@
 			)
 		)
-		(property "url" "https://www.digikey.com/product-detail/en/yageo/RC0603JR-072K2L/311-2.2KGRCT-ND/729676"
+		(property "URL" "https://www.digikey.com/en/products/detail/yageo/AC0603JR-072K2L/5896418"
 			(at 213.36 170.18 90)
 			(effects
@@
 			)
 		)
-		(property "url" "https://www.digikey.com/product-detail/en/yageo/RC0603JR-072K2L/311-2.2KGRCT-ND/729676"
+		(property "URL" "https://www.digikey.com/en/products/detail/yageo/AC0603JR-072K2L/5896418"
 			(at 213.36 88.9 90)
 			(effects
@@
 	)
 	(symbol
+		(lib_id "Device:R")
+		(at 95.25 127 0)
+		(unit 1)
+		(exclude_from_sim no)
+		(in_bom yes)
+		(on_board yes)
+		(dnp no)
+		(property "Reference" "R1"
+			(at 97.282 127 90)
+			(effects
+				(font
+					(size 1.27 1.27)
+				)
+			)
+		)
+		(property "Value" "10k 5%"
+			(at 92.964 127 90)
+			(effects
+				(font
+					(size 1.27 1.27)
+				)
+			)
+		)
+		(property "Footprint" "Capacitor_SMD:C_0603_1608Metric"
+			(at 93.472 127 90)
+			(effects
+				(font
+					(size 1.27 1.27)
+				)
+				(hide yes)
+			)
+		)
+		(property "Datasheet" "~"
+			(at 95.25 127 0)
+			(effects
+				(font
+					(size 1.27 1.27)
+				)
+				(hide yes)
+			)
+		)
+		(property "Description" "Resistor"
+			(at 95.25 127 0)
+			(effects
+				(font
+					(size 1.27 1.27)
+				)
+				(hide yes)
+			)
+		)
+		(property "URL" "https://www.digikey.com/product-detail/en/yageo/RC0603JR-072K2L/311-2.2KGRCT-ND/729676"
+			(at 95.25 127 90)
+			(effects
+				(font
+					(size 1.524 1.524)
+				)
+				(hide yes)
+			)
+		)
+		(pin "2"
+		)
+		(pin "1"
+		)
+		(instances
+			(project "multi_sensor_host"
+				(path "/895fe915-d6d4-4da2-a6ec-6414a345dc15/46e9a6e6-b007-46d9-9be8-93a48bc459dd"
+					(reference "R1")
+					(unit 1)
+				)
+				(path "/895fe915-d6d4-4da2-a6ec-6414a345dc15/4b2528f7-9d95-4490-9078-a08d5cbf26f8"
+					(reference "R4")
+					(unit 1)
+				)
+			)
+		)
+	)
+	(symbol
 		(lib_id "Device:C")
 		(at 190.5 91.44 0)
@@
 			)
 		)
-		(property "url" "https://www.digikey.com/product-detail/en/samsung-electro-mechanics-america-inc/CL10B475KQ8NQNC/1276-2087-1-ND/3890173"
+		(property "URL" "https://www.digikey.com/product-detail/en/samsung-electro-mechanics-america-inc/CL10B475KQ8NQNC/1276-2087-1-ND/3890173"
 			(at 190.5 91.44 0)
 			(effects
@@
 			)
 		)
-		(property "url" "https://www.digikey.com/product-detail/en/yageo/RC0603JR-072K2L/311-2.2KGRCT-ND/729676"
+		(property "URL" "https://www.digikey.com/en/products/detail/yageo/AC0603JR-072K2L/5896418"
 			(at 224.79 149.86 90)
 			(effects
@@
 			)
 		)
-		(property "url" "https://www.digikey.com/product-detail/en/yageo/RC0603JR-072K2L/311-2.2KGRCT-ND/729676"
+		(property "URL" "https://www.digikey.com/en/products/detail/yageo/AC0603JR-072K2L/5896418"
 			(at 224.79 170.18 90)
 			(effects
@@
 			)
 		)
-		(property "url" "https://www.digikey.com/product-detail/en/yageo/RC0603JR-072K2L/311-2.2KGRCT-ND/729676"
+		(property "URL" "https://www.digikey.com/en/products/detail/yageo/AC0603JR-072K2L/5896418"
 			(at 224.79 190.5 90)
 			(effects

Commit message: Placing components, tracing wires.
Parts:
- removed C11: 100n, Capacitor_SMD:C_0603_1608Metric, symbol Device:C
- removed R1: 10k 5%, Capacitor_SMD:C_0603_1608Metric, symbol Device:R
Connections:
- net rst: now reaches U1.3 (~{RESET})
