File: schematics/multi_sensor_host/tca9548a_sheet.kicad_sch (KiCad schematic)
At the start: 21 parts, among them U1 TCA9548A_TSSOP

Commit message: All I2C multiplexers have the same address selection pins configuration. Added 22u capacitors.
Parts:
- C2: value 4u7 -> 22u; URL https://www.digikey.com/product-detail/en/samsung-electro-m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 -> https://www.digikey.com/en/products/detail/kyocera-avx/0603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
Changed lines of the file:
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@@
+	)
+	(symbol
+		(lib_id "Device:C")
+		(at 190.5 91.44 0)
+		(unit 1)
+		(exclude_from_sim no)
+		(in_bom yes)
+		(on_board yes)
+		(dnp no)
+		(property "Reference" "C2"
+			(at 191.135 88.9 0)
+			(effects
+				(font
+					(size 1.27 1.27)
+				)
+				(justify left)
+			)
+		)
+		(property "Value" "22u"
+			(at 191.135 93.98 0)
+			(effects
+				(font
+					(size 1.27 1.27)
+				)
+				(justify left)
+			)
+		)
+		(property "Footprint" "Capacitor_SMD:C_0603_1608Metric"
+			(at 191.4652 95.25 0)
+			(effects
+				(font
+					(size 1.27 1.27)
+				)
+				(hide yes)
+			)
+		)
+		(property "Datasheet" "~"
+			(at 190.5 91.44 0)
+			(effects
+				(font
+					(size 1.27 1.27)
+				)
+				(hide yes)
+			)
+		)
+		(property "Description" "Unpolarized capacitor"
+			(at 190.5 91.44 0)
+			(effects
+				(font
+					(size 1.27 1.27)
+				)
+				(hide yes)
+			)
+		)
+		(property "URL" "https://www.digikey.com/en/products/detail/kyocera-avx/0603YD226MAT2A/17866383"
+			(at 190.5 91.44 0)
+			(effects
+				(font
+					(size 1.524 1.524)
+				)
+				(hide yes)
+			)
+		)
+		(pin "1"
+		)
+		(pin "2"
+		)
+		(instances
+			(project "multi_sensor_host"
+				(path "/895fe915-d6d4-4da2-a6ec-6414a345dc15/46e9a6e6-b007-46d9-9be8-93a48bc459dd"
+					(reference "C2")
+					(unit 1)
+				)
+				(path "/895fe915-d6d4-4da2-a6ec-6414a345dc15/4b2528f7-9d95-4490-9078-a08d5cbf26f8"
+					(reference "C12")
+					(unit 1)
+				)
+				(path "/895fe915-d6d4-4da2-a6ec-6414a345dc15/9e1e7fd2-4492-4d4c-9b2e-cc16e85c9a24"
+					(reference "C14")
+					(unit 1)
+				)
+			)
+		)
 	)
 	(symbol
@@
 					(unit 1)
 				)
-			)
-		)
-	)
-	(symbol
-		(lib_id "Device:C")
-		(at 190.5 91.44 0)
-		(unit 1)
-		(exclude_from_sim no)
-		(in_bom yes)
-		(on_board yes)
-		(dnp no)
-		(property "Reference" "C2"
-			(at 191.135 88.9 0)
-			(effects
-				(font
-					(size 1.27 1.27)
-				)
-				(justify left)
-			)
-		)
-		(property "Value" "4u7"
-			(at 191.135 93.98 0)
-			(effects
-				(font
-					(size 1.27 1.27)
-				)
-				(justify left)
-			)
-		)
-		(property "Footprint" "Capacitor_SMD:C_0603_1608Metric"
-			(at 191.4652 95.25 0)
-			(effects
-				(font
-					(size 1.27 1.27)
-				)
-				(hide yes)
-			)
-		)
-		(property "Datasheet" "~"
-			(at 190.5 91.44 0)
-			(effects
-				(font
-					(size 1.27 1.27)
-				)
-				(hide yes)
-			)
-		)
-		(property "Description" "Unpolarized capacitor"
-			(at 190.5 91.44 0)
-			(effects
-				(font
-					(size 1.27 1.27)
-				)
-				(hide yes)
-			)
-		)
-		(property "URL" "https://www.digikey.com/product-detail/en/samsung-electro-mechanics-america-inc/CL10B475KQ8NQNC/1276-2087-1-ND/3890173"
-			(at 190.5 91.44 0)
-			(effects
-				(font
-					(size 1.524 1.524)
-				)
-				(hide yes)
-			)
-		)
-		(pin "2"
-		)
-		(pin "1"
-		)
-		(instances
-			(project "multi_sensor_host"
-				(path "/895fe915-d6d4-4da2-a6ec-6414a345dc15/46e9a6e6-b007-46d9-9be8-93a48bc459dd"
-					(reference "C2")
-					(unit 1)
-				)
-				(path "/895fe915-d6d4-4da2-a6ec-6414a345dc15/4b2528f7-9d95-4490-9078-a08d5cbf26f8"
-					(reference "C14")
-					(unit 1)
-				)
-				(path "/895fe915-d6d4-4da2-a6ec-6414a345dc15/9e1e7fd2-4492-4d4c-9b2e-cc16e85c9a24"
-					(reference "C12")
-					(unit 1)
-				)
