File: schematics/multi_sensor_host/multi_sensor_host.kicad_pcb (KiCad board)
At the start: 2 copper layers, 169 parts, among them J1 left hand 0, J10 swd, J11 stm_boot, J13 right hand 0, J14 right hand 1, J15 right hand 2, J16 right hand 3, J17 rst_mcu, J18 left hand 3, J19 left leg 0, J2 left hand 1, J20 left leg 1, J21 right lef 0, J22 right leg 1, J3 bm_cfg, J4 left hand 2, J5 tx, J6 MY_USB_B, J7 rst_bm71, J8 rx, J9 uart1, U1 TCA9548A_TSSOP, U11 MCP111, U12 BM71BLES1FC2-0B02AA, U2 TCA9548A_TSSOP, U3 TCA9548A_TSSOP, U4 MCP111, U5 TPS79333-EP, U8 MCP73812, U9 MCP1603, Y1 Crystal

Commit message: a
Parts:
- moved R45 363.9 mm to (285.5, -53.7), turned to 90 degrees
- moved R44 361.4 mm to (291.5, -53.7), turned to 90 degrees
- moved R54 358.6 mm to (275.0, -53.7), turned to 90 degrees
- moved R55 356.0 mm to (270.5, -53.7), turned to 90 degrees
- moved R46 354.3 mm to (272.5, -53.7), turned to 90 degrees
- moved R52 349.9 mm to (293.5, -53.7)
- moved R53 347.6 mm to (289.0, -53.7), turned to 90 degrees
- moved R47 341.4 mm to (267.0, -53.7), turned to 90 degrees
- moved R49 339.1 mm to (252.0, -53.7), turned to 90 degrees
- moved R48 334.0 mm to (256.5, -53.7), turned to 90 degrees
- moved R40 327.0 mm to (254.0, -53.7), turned to 90 degrees
- moved R41 325.8 mm to (249.0, -53.7), turned to 90 degrees
- moved C77 320.9 mm to (283.0, -53.7), turned to -90 degrees
- moved C76 318.2 mm to (281.0, -53.7), turned to -90 degrees
- moved C73 310.7 mm to (264.5, -53.7), turned to -90 degrees
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
Commit message: a
Parts:
- moved R2 14.6 mm to (43.6, -45.9), turned to 180 degrees
- moved C2 14.4 mm to (39.3, -49.7), turned to 180 degrees
- moved R3 13.6 mm to (43.6, -44.4), turned to 180 degrees
- moved C1 11.9 mm to (39.3, -47.6), turned to 180 degrees
- moved U1 3.94 mm to (37.1, -42.0), turned to 0 degrees

Commit message: a
Parts:
- moved C40 38.9 mm to (-0.76, -54.7)
- moved C41 38.9 mm to (1.24, -54.7)
- moved C44 38.9 mm to (17.8, -54.7)
- moved C45 38.9 mm to (19.7, -54.7)
- moved J18 38.9 mm to (11.2, -63.1)
- moved J4 38.9 mm to (29.7, -63.1)
- moved R14 38.9 mm to (27.6, -54.7)
- moved R15 38.9 mm to (22.0, -54.7)
- moved R16 38.9 mm to (9.04, -54.7)
- moved R17 38.9 mm to (3.64, -54.7)
- moved R22 38.9 mm to (29.7, -54.7)
- moved R23 38.9 mm to (25.4, -54.7)
- moved R24 38.9 mm to (11.2, -54.7)
- moved R25 38.9 mm to (6.94, -54.7)
- moved C56 37.5 mm to (163.3, -53.6)
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
Commit message: a
Parts:
- TP1, TP2: footprint Connector_PinHeader_1.00mm:PinHeader_1x01_P1.00mm_Vertical -> Connector_Pin:Pin_D1.4mm_L8.5mm_W2.8mm_FlatFork
- moved C33 253.3 mm to (132.3, 53.6), turned to -90 degrees
- moved C16 250.8 mm to (130.3, 53.6), turned to -90 degrees
- moved C34 248.9 mm to (132.0, 56.3), turned to 180 degrees
- moved R86 246.6 mm to (138.7, 50.5), turned to -90 degrees
- moved U12 246.1 mm to (124.0, 51.5), turned to 0 degrees
- moved C10 245.9 mm to (132.0, 58.3), turned to 180 degrees
- moved J3 242.3 mm to (136.0, 51.0), turned to 0 degrees
- moved C22 241.9 mm to (138.7, 53.8), turned to -90 degrees
- moved D5 239.2 mm to (128.9, 60.6), turned to -90 degrees
- moved J13 234.3 mm to (71.8, 148.7), turned to 0 degrees
- moved J5 231.3 mm to (124.5, 61.0), turned to 0 degrees
- moved R98 231.2 mm to (129.0, 66.2), turned to 90 degrees
- moved J8 226.2 mm to (120.5, 61.0), turned to 0 degrees
- moved R31 220.5 mm to (71.3, 140.6), turned to -90 degrees
- moved J14 220.5 mm to (90.3, 148.7), turned to 0 degrees
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
Commit message: a
Parts:
- moved D4 253.8 mm to (108.0, 68.2)
- moved R92 253.8 mm to (104.5, 69.7)
- moved D3 239.0 mm to (108.0, 80.6)
- moved R90 239.0 mm to (104.5, 81.8)
- moved D6 233.2 mm to (108.0, 74.5)
- moved R89 233.2 mm to (104.5, 75.8)
- moved C15 210.3 mm to (122.7, 69.0)
- moved J7 210.3 mm to (126.0, 75.5)
- moved R57 210.3 mm to (126.3, 69.0)
- moved U4 210.3 mm to (124.8, 72.0)
- moved J10 187.7 mm to (77.0, 74.1), turned to 180 degrees
- moved R93 187.3 mm to (93.3, 64.2), turned to 180 degrees
- moved J9 185.9 mm to (92.0, 67.0), turned to 90 degrees
- moved C21 180.5 mm to (102.6, 87.2)
- moved R94 180.5 mm to (101.0, 90.4)
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
Commit message: a
Parts:
- moved C40 36.6 mm to (84.9, 131.4)
- moved C41 36.6 mm to (84.9, 129.4)
- moved R2 36.6 mm to (98.9, 125.4)
- moved U1 36.6 mm to (95.0, 119.0)
- moved C1 36.6 mm to (100.6, 121.2)
- moved C19 36.6 mm to (84.9, 94.4)
- moved C2 36.6 mm to (102.7, 121.2)
- moved C20 36.6 mm to (84.9, 92.4)
- moved C36 36.6 mm to (84.9, 75.9)
- moved C37 36.6 mm to (84.9, 73.9)
- moved C44 36.6 mm to (84.9, 112.8)
- moved C45 36.6 mm to (84.9, 110.9)
- moved J1 36.6 mm to (76.5, 63.8)
- moved J18 36.6 mm to (76.5, 119.4)
- moved J2 36.6 mm to (76.5, 82.4)
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
Commit message: a
Parts:
- moved R31 37.2 mm to (102.4, 133.2), turned to 180 degrees
- moved R7 34.4 mm to (102.4, 135.2), turned to 180 degrees
- moved R32 31.3 mm to (102.4, 137.2), turned to 180 degrees
- moved R30 29.7 mm to (121.8, 133.7), turned to 0 degrees
- moved R8 27.2 mm to (102.4, 139.2), turned to 180 degrees
- moved R38 25.9 mm to (121.8, 135.7), turned to 0 degrees
- moved C1 25.2 mm to (75.4, 121.2)
- moved C2 25.2 mm to (77.6, 121.2)
- moved R2 25.2 mm to (73.8, 125.4)
- moved U1 25.2 mm to (69.9, 119.0)
- moved C19 25.2 mm to (59.8, 94.4)
- moved C20 25.2 mm to (59.8, 92.4)
- moved C36 25.2 mm to (59.8, 75.9)
- moved C37 25.2 mm to (59.8, 73.9)
- moved C40 25.2 mm to (59.8, 131.3)
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
Commit message: a
Parts:
- moved C32 62.6 mm to (95.6, 129.3)
- moved J17 62.6 mm to (98.3, 136.3)
- moved R97 62.6 mm to (99.1, 129.3)
- moved U11 62.6 mm to (97.3, 132.5)
- moved C15 50.6 mm to (106.2, 117.5)
- moved J7 50.6 mm to (109.5, 124.0)
- moved R57 50.6 mm to (109.7, 117.5)
- moved U4 50.6 mm to (108.2, 120.5)
- moved R18 46.6 mm to (88.3, 100.6)
- moved C72 46.6 mm to (128.5, 99.5)
- moved C73 46.6 mm to (128.5, 101.5)
- moved R10 46.4 mm to (88.3, 102.6)
- moved R19 46.3 mm to (88.3, 104.6)
- moved R47 46.2 mm to (128.5, 103.5)
- moved R11 45.2 mm to (88.3, 106.6)
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Other:
- copper layers 2 -> 4
