File: schematics/board_bmi085/board_bmi085/board_bmi085.kicad_sch (KiCad schematic)
At the start: 17 parts, among them J1 Conn_01x08_Pin, J3 Conn_01x08_Pin

Commit message: a
Parts:
- R1, R2, R3, R4: footprint Resistor_SMD:R_0603_1608Metric -> Resistor_SMD:R_0402_1005Metric
Changed lines of the file:
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@@
 			)
 		)
-		(property "Footprint" "Resistor_SMD:R_0603_1608Metric"
+		(property "Footprint" "Resistor_SMD:R_0402_1005Metric"
 			(at 42.672 46.99 90)
 			(effects
@@
 			)
 		)
-		(property "Footprint" "Resistor_SMD:R_0603_1608Metric"
+		(property "Footprint" "Resistor_SMD:R_0402_1005Metric"
 			(at 42.672 88.9 90)
 			(effects
@@
 			)
 		)
-		(property "Footprint" "Resistor_SMD:R_0603_1608Metric"
+		(property "Footprint" "Resistor_SMD:R_0402_1005Metric"
 			(at 42.672 101.6 90)
 			(effects
@@
 			)
 		)
-		(property "Footprint" "Resistor_SMD:R_0603_1608Metric"
+		(property "Footprint" "Resistor_SMD:R_0402_1005Metric"
 			(at 42.672 59.69 90)
 			(effects

Commit message: Re-done the sensor board. Now it can be up 4 sensors on a single cable.
Parts:
- removed R10, R11, R9: 100, Capacitor_SMD:C_0402_1005Metric, symbol Device:R
- removed R12, R13: 100, Resistor_SMD:R_0603_1608Metric, symbol Device:R
- removed R14, R15: 2k, Resistor_SMD:R_0603_1608Metric, symbol Device:R
- added R5, R6, R7: 0, Resistor_SMD:R_0402_1005Metric, symbol Device:R
- R1, R2, R3, R4: value 10k -> 0
- R8: value 100 -> 0; footprint Capacitor_SMD:C_0402_1005Metric -> Resistor_SMD:R_0402_1005Metric; url https://www.digikey.com/en/products/detail/yageo/AC0603JR-0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 -> https://www.digikey.com/en/products/detail/yageo/RC0603JR-1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
Connections:
- net scl: now also R5.2, R6.2; no longer J1.3 (Pin_3), J3.3 (Pin_3)
- net sda: now also R8.2, R7.2; no longer J1.1 (Pin_1), J3.1 (Pin_1)
- net at U1.16 (INT1): no longer R8.1
- net int_a renamed sda_b
- net sda_b: now also R8.1
- net int_b renamed scl_b
- net scl_b: now also R5.1
- new net scl_a: J1.3 (Pin_3), J3.3 (Pin_3), R6.1
- new net sda_a: J1.1 (Pin_1), J3.1 (Pin_1), R7.1
- no-connect marks 2 -> 6
Other:
- note removed: "Here at most one pin should be connected to at most one line"
- note removed: "These might not me needed. There are already pullups on the main board."
- moved on the sheet: C1, C2, U1
